Commit message: feat: rename package to Ranger + robot redesign + stack tuning
## Package Rename
- Renamed package from def_bot to Ranger
- Updated all references in CMakeLists.txt and package.xml

## URDF Restructure
- Renamed urdf/ folder to description/
- Split monolithic xacro into separate files:
  - amr_core.xacro      (chassis + wheel geometry)
  - amr.urdf.xacro      (top-level robot file)
  - sensors.xacro       (LiDAR + IMU sensor links)
  - controls.xacro      (ros2_control hardware interface)
  - gazebo.xacro        (Gazebo plugins + material props)
  - materials.xacro     (RViz visual materials)

## Robot Redesign
- Wheel radius: 80mm → 90mm
- Caster wheel radius: 10mm → 15mm
- Caster assembly: joined to base_link via new_body joint
- Wheel separation: 0.35m → 0.205m
- Wheel radius param: 0.1 → 0.045m

## Controller Tuning (controller.yaml)
- enable_odom_tf: true
- wheel_separation: 0.35 → 0.205
- wheel_radius: 0.1 → 0.045

## EKF Tuning (ekf.yaml)
- Added publish_odom_to_base_link: true

## SLAM Tuning (mapper_params_online_async.yaml)
- Added publish_map_to_odom_tf: true
- Added tf_buffer_duration: 30.0

## Launch File (gz_sim.launch.py)
- Merged all bridges into single ros_gz_bridge node:
  /scan, /imu, /clock, /laserscan, /pointcloud
- Added 2s delay before EKF node starts

File: description/def_new_bot_final.xacro (robot description, xacro)
@@ -1,6 +1,4 @@
-<?xml version="1.0" ?>
+<!-- <?xml version="1.0" ?>
 <robot name="AMR" xmlns:xacro="http://www.ros.org/wiki/xacro">
-  <xacro:include filename="$(find def_bot)/urdf/def_bot_materials.xacro" />
-  <xacro:include filename="$(find def_bot)/urdf/def_bot_gazebo.xacro" />
   <!-- <link name="base_footprint"/>
   <joint name="base_joint" type="fixed">
@@ -18,5 +16,5 @@
         <origin xyz="0 0 0" rpy="0 0 0"/>
         <geometry>
-          <mesh filename="package://def_bot/meshes/base_link.stl" scale="0.001 0.001 0.001"/>
+          <mesh filename="package://ranger/meshes/base_link.stl" scale="0.001 0.001 0.001"/>
         </geometry>
         <material name="silver"/>
@@ -25,5 +23,5 @@
         <origin xyz="0 0 0" rpy="0 0 0"/>
         <geometry>
-          <mesh filename="package://def_bot/meshes/base_link.stl" scale="0.001 0.001 0.001"/>
+          <mesh filename="package://ranger/meshes/base_link.stl" scale="0.001 0.001 0.001"/>
         </geometry>
       </collision>
@@ -38,5 +36,5 @@
         <origin xyz="0.055 0.1025 -0.04" rpy="0 0 0"/>
         <geometry>
-          <mesh filename="package://def_bot/meshes/right_wheel_link_1.stl" scale="0.001 0.001 0.001"/>
+          <mesh filename="package://ranger/meshes/right_wheel_link_1.stl" scale="0.001 0.001 0.001"/>
         </geometry>
         <material name="silver"/>
@@ -45,5 +43,5 @@
         <origin xyz="0.055 0.1025 -0.04" rpy="0 0 0"/>
         <geometry>
-          <mesh filename="package://def_bot/meshes/right_wheel_link_1.stl" scale="0.001 0.001 0.001"/>
+          <mesh filename="package://ranger/meshes/right_wheel_link_1.stl" scale="0.001 0.001 0.001"/>
         </geometry>
       </collision>
@@ -58,5 +56,5 @@
         <origin xyz="0.055 -0.1025 -0.04" rpy="0 0 0"/>
         <geometry>
-          <mesh filename="package://def_bot/meshes/left_wheel_link_1.stl" scale="0.001 0.001 0.001"/>
+          <mesh filename="package://ranger/meshes/left_wheel_link_1.stl" scale="0.001 0.001 0.001"/>
         </geometry>
         <material name="silver"/>
@@ -65,5 +63,5 @@
         <origin xyz="0.055 -0.1025 -0.04" rpy="0 0 0"/>
         <geometry>
-          <mesh filename="package://def_bot/meshes/left_wheel_link_1.stl" scale="0.001 0.001 0.001"/>
+          <mesh filename="package://ranger/meshes/left_wheel_link_1.stl" scale="0.001 0.001 0.001"/>
         </geometry>
       </collision>
@@ -78,5 +76,5 @@
         <origin xyz="-0.05 -0.0 -0.105" rpy="0 0 0"/>
         <geometry>
-          <mesh filename="package://def_bot/meshes/lidar_link_1.stl" scale="0.001 0.001 0.001"/>
+          <mesh filename="package://ranger/meshes/lidar_link_1.stl" scale="0.001 0.001 0.001"/>
         </geometry>
         <material name="silver"/>
@@ -85,5 +83,5 @@
         <origin xyz="-0.05 -0.0 -0.105" rpy="0 0 0"/>
         <geometry>
-          <mesh filename="package://def_bot/meshes/lidar_link_1.stl" scale="0.001 0.001 0.001"/>
+          <mesh filename="package://ranger/meshes/lidar_link_1.stl" scale="0.001 0.001 0.001"/>
         </geometry>
       </collision>
@@ -106,25 +104,25 @@
       <child link="lidar_link_1"/>
     </joint>
-    <ros2_control name="DiffDriveSystem" type="system">
-            <hardware>
+            <ros2_control name="DiffDriveSystem" type="system">
+              <hardware>
                 <plugin>ign_ros2_control/IgnitionSystem</plugin>
               <!-- <plugin>gz_ros2_control/GazeboSimSystem</plugin> -->
-            </hardware>
-            <joint name="left_wheel_joint">
+              </hardware>
+              <joint name="left_wheel_joint">
                 <command_interface name="velocity"/>
                 <state_interface name="position"/>
                 <state_interface name="velocity"/>
-            </joint>
-            <joint name="right_wheel_joint">
+              </joint>
+              <joint name="right_wheel_joint">
                 <command_interface name="velocity"/>
                 <state_interface name="position"/>
                 <state_interface name="velocity"/>
-            </joint>
-        </ros2_control>
+              </joint>
+            </ros2_control>
       <!-- <gazebo>
             <plugin filename="libign_ros2_control-system.so"
                     name="ign_ros2_control::IgnitionROS2ControlPlugin">
-                <parameters>$(find def_bot)/config/controller.yaml</parameters>
+                <parameters>$(find ranger)/config/controller.yaml</parameters>
             </plugin>
       </gazebo> -->
-</robot>
+</robot> -->

File: description/gazebo.xacro (robot description, xacro)
@@ -2,29 +2,39 @@
 <robot name="Diff_drive_robot" xmlns:xacro="http://www.ros.org/wiki/xacro" >
 <xacro:property name="body_color" value="Gazebo/Silver" />
-        <gazebo reference="base_link">
-          <material>${body_color}</material>
-          <mu1>0.2</mu1>
-          <mu2>0.2</mu2>
-          <selfCollide>true</selfCollide>
-          <gravity>true</gravity>
-        </gazebo>
-        <gazebo reference="left_wheel_1">
-          <material>${body_color}</material>
-          <mu1>0.2</mu1>
-          <mu2>0.2</mu2>
-          <selfCollide>true</selfCollide>
-        </gazebo>
-        <gazebo reference="right_wheel_1">
-          <material>${body_color}</material>
-          <mu1>0.2</mu1>
-          <mu2>0.2</mu2>
-          <selfCollide>true</selfCollide>
-        </gazebo>
-        <gazebo reference="lidar_link_1">
-          <material>${body_color}</material>
-          <mu1>0.2</mu1>
-          <mu2>0.2</mu2>
-          <selfCollide>true</selfCollide>
-        </gazebo>
+  <gazebo reference="base_link">
+    <material>${body_color}</material>
+    <mu1>0.2</mu1>
+    <mu2>0.2</mu2>
+    <selfCollide>true</selfCollide>
+    <gravity>true</gravity>
+  </gazebo>
+  <gazebo reference="left_wheel_1">
+    <material>${body_color}</material>
+    <mu1>2.0</mu1>
+    <mu2>2.0</mu2>
+    <kp>1000000.0</kp>
+    <kd>100.0</kd>
+    <selfCollide>true</selfCollide>
+  </gazebo>
+  <gazebo reference="right_wheel_1">
+    <material>${body_color}</material>
+    <mu1>2.0</mu1>
+    <mu2>2.0</mu2>
+    <kp>1000000.0</kp>
+    <kd>100.0</kd>
+    <selfCollide>true</selfCollide>
+  </gazebo>
+  <gazebo reference="lidar_link_1">
+    <material>${body_color}</material>
+    <mu1>0.2</mu1>
+    <mu2>0.2</mu2>
+    <selfCollide>true</selfCollide>
+  </gazebo>
+  <gazebo reference="castor_wheel_link_1">
+    <material>${body_color}</material>
+    <mu1>0.0</mu1>
+    <mu2>0.0</mu2>
+    <selfCollide>true</selfCollide>
+  </gazebo>
       <!-- <plugin filename="ignition-gazebo-joint-state-publisher-system" name="ignition::gazebo::systems::JointStatePublisher">
         <update_rate>10</update_rate>
@@ -35,31 +45,31 @@
               name="ign_ros2_control::IgnitionROS2ControlPlugin"> -->
     <!-- <plugin filename="gz_ros2_control-system" name="gz_ros2_control::GazeboSimROS2ControlPlugin"> -->
-  <gazebo reference="lidar_link_1">
+  <!-- <gazebo reference="lidar_link_1">
     <sensor name="lidar" type="gpu_lidar">
-        <topic>/scan</topic>
-        <update_rate>5</update_rate>
-        <gz_frame_id>lidar_link_1</gz_frame_id>
-        <ray>
-          <scan>
-            <horizontal>
-              <samples>360</samples>
-              <resolution>1</resolution>
-              <min_angle>-3.14159</min_angle>
-              <max_angle>3.14159</max_angle>
-            </horizontal>
-          </scan>
-          <range>
-            <min>0.35</min>
-            <max>10.0</max>
-            <resolution>0.01</resolution>
-          </range>
-          <noise>
-            <type>gaussian</type>
-            <mean>0.0</mean>
-            <stddev>0.01</stddev>
-          </noise>
-        </ray>
-        <always_on>true</always_on>
-        <visualize>true</visualize>
+      <topic>/scan</topic>
+      <update_rate>5</update_rate>
+      <gz_frame_id>lidar_link_1</gz_frame_id>
+      <ray>
+        <scan>
+          <horizontal>
+            <samples>360</samples>
+            <resolution>1</resolution>
+            <min_angle>-3.14159</min_angle>
+            <max_angle>3.14159</max_angle>
+          </horizontal>
+        </scan>
+        <range>
+          <min>0.35</min>
+          <max>10.0</max>
+          <resolution>0.01</resolution>
+        </range>
+        <noise>
+          <type>gaussian</type>
+          <mean>0.0</mean>
+          <stddev>0.005</stddev>
+        </noise>
+      </ray>
+      <always_on>true</always_on>
+      <visualize>true</visualize>
     </sensor>
   </gazebo>
@@ -114,15 +124,9 @@
       <visualize>false</visualize>
     </sensor>
-  </gazebo>
-  <gazebo>
-      <plugin filename="ign_ros2_control-system" name="ign_ros2_control::IgnitionROS2ControlPlugin">
-        <parameters>$(find def_bot)/config/controller.yaml</parameters>
-      </plugin>
-  </gazebo>
-  <gazebo>
-    <plugin filename="ignition-gazebo-sensors-system"
-            name="ignition::gazebo::systems::Sensors">
-      <render_engine>ogre</render_engine>
+  </gazebo> -->
+  <!-- <gazebo>
+    <plugin filename="ign_ros2_control-system" name="ign_ros2_control::IgnitionROS2ControlPlugin">
+      <parameters>$(find ranger)/config/controller.yaml</parameters>
     </plugin>
-  </gazebo>
+  </gazebo> -->
 </robot>

File: description/materials.xacro (robot description, xacro)
@@ -1,6 +1,6 @@
 <?xml version="1.0" ?>
 <robot name="Diff_drive_robot" xmlns:xacro="http://www.ros.org/wiki/xacro" >
-<material name="silver">
-  <color rgba="0.700 0.700 0.700 1.000"/>
-</material>
+  <material name="silver">
+    <color rgba="0.700 0.700 0.700 1.000"/>
+  </material>
 </robot>
